Commit message: Imported upstream version '0.3.3' of 'upstream'

File: bwi_gazebo_entities/gazebo/controllable_person.gazebo.xacro (robot description, xacro)
@@ -9,12 +9,12 @@
         <update_rate>20.0</update_rate>
         <camera>
-          <horizontal_fov>1.0</horizontal_fov>
+          <horizontal_fov>0.5</horizontal_fov>
           <image>
-            <width>640</width>
+            <width>320</width>
             <height>480</height>
             <format>R8G8B8</format>
           </image>
           <clip>
-            <near>0.01</near>
+            <near>1.75</near>
             <far>30.0</far>
           </clip>

File: bwi_gazebo_entities/urdf/person.urdf.xacro (robot description, xacro)
@@ -39,5 +39,5 @@
     </link>
     <gazebo reference="base_link">
-      <material>Gazebo/Black</material>
+      <material>Gazebo/White</material>
     </gazebo>
     <!-- depth perception lidar -->
@@ -75,9 +75,9 @@
           <cylinder length="0.9" radius="0.09" />
         </geometry>
-        <material name="black" />
+        <material name="light_grey" />
       </visual>
     </link>
     <gazebo reference="left_leg_link">
-      <material>Gazebo/Black</material>
+      <material>Gazebo/White</material>
     </gazebo>
     <xacro:default_surface name="left_leg" />
@@ -101,9 +101,9 @@
           <cylinder length="0.9" radius="0.09" />
         </geometry>
-        <material name="black" />
+        <material name="light_grey" />
       </visual>
     </link>
     <gazebo reference="right_leg_link">
-      <material>Gazebo/Black</material>
+      <material>Gazebo/White</material>
     </gazebo>
     <xacro:default_surface name="right_leg" />
@@ -126,21 +126,21 @@
           <sphere radius="0.15" />
         </geometry>
-        <material name="black" />
+        <material name="light_grey" />
       </visual>
     </link>
     <gazebo reference="head_link">
-      <material>Gazebo/Black</material>
+      <material>Gazebo/White</material>
     </gazebo>
     <!-- camera -->
-    <joint name="camera_joint" type="fixed">
-      <origin xyz="0.151 0 0" rpy="0 ${M_PI/12} 0" />
-      <parent link="head_link"/>
-      <child link="camera_link" />
-    </joint>
     <!-- <joint name="camera_joint" type="fixed"> -->
-    <!--   <origin xyz="-1.0 0 0.25" rpy="0 ${M_PI/12} 0" /> -->
+    <!--   <origin xyz="0.151 0 0" rpy="0 ${M_PI/12} 0" /> -->
     <!--   <parent link="head_link"/> -->
     <!--   <child link="camera_link" /> -->
     <!-- </joint> -->
+    <joint name="camera_joint" type="fixed">
+      <origin xyz="-2 0 0.75" rpy="0 ${M_PI/8} 0" />
+      <parent link="head_link"/>
+      <child link="camera_link" />
+    </joint>
     <link name="camera_link">
       <inertial>
@@ -186,9 +186,9 @@
           <cylinder length="0.35" radius="0.07" />
         </geometry>
-        <material name="black" />
+        <material name="light_grey" />
       </visual>
     </link>
     <gazebo reference="left_arm_link">
-      <material>Gazebo/Black</material>
+      <material>Gazebo/White</material>
     </gazebo>
     <!-- left fore arm -->
@@ -211,9 +211,9 @@
           <cylinder length="0.35" radius="0.07" />
         </geometry>
-        <material name="black" />
+        <material name="light_grey" />
       </visual>
     </link>
     <gazebo reference="left_forearm_link">
-      <material>Gazebo/Black</material>
+      <material>Gazebo/White</material>
     </gazebo>
     <!-- right arm -->
@@ -236,9 +236,9 @@
           <cylinder length="0.35" radius="0.07" />
         </geometry>
-        <material name="black" />
+        <material name="light_grey" />
       </visual>
     </link>
     <gazebo reference="right_arm_link">
-      <material>Gazebo/Black</material>
+      <material>Gazebo/White</material>
     </gazebo>
     <!-- right fore arm -->
@@ -261,9 +261,9 @@
           <cylinder length="0.35" radius="0.07" />
         </geometry>
-        <material name="black" />
+        <material name="light_grey" />
       </visual>
     </link>
     <gazebo reference="right_forearm_link">
-      <material>Gazebo/Black</material>
+      <material>Gazebo/White</material>
     </gazebo>
     <gazebo>
